File: HW4/HW4/HW4.kicad_pcb (KiCad board)
At the start: 2 copper layers, 50 x 50 mm, 4 parts, among them U1 AP7384-33V

Commit message: HW4 Done lawl
Parts:
- added C2: 1uF, Capacitor_THT:C_Disc_D5.1mm_W3.2mm_P5.00mm, F.Cu at (141.2, 84.8)
- added C3: 1uF, Capacitor_THT:C_Disc_D5.1mm_W3.2mm_P5.00mm, F.Cu at (141.2, 80.3)
- added C4: 0.1uF, Capacitor_THT:C_Disc_D3.4mm_W2.1mm_P2.50mm, F.Cu at (112.8, 77.7)
- added C5: 0.1uF, Capacitor_THT:C_Disc_D3.4mm_W2.1mm_P2.50mm, F.Cu at (132.1, 61.0)
- added C6: 1uF, Capacitor_THT:C_Disc_D5.1mm_W3.2mm_P5.00mm, F.Cu at (132.1, 79.8)
- added D2: YELLOW, LED_THT:LED_D3.0mm, F.Cu at (138.2, 90.7)
- added D3: GREEN, LED_THT:LED_D3.0mm, F.Cu at (141.2, 98.3)
- added J1: CP2102, Connector_PinSocket_2.54mm:PinSocket_1x06_P2.54mm_Vertical, F.Cu at (110.2, 52.8)
- added J2: Battery, Connector_PinSocket_2.54mm:PinSocket_1x02_P2.54mm_Vertical, F.Cu at (103.6, 55.9)
- added J3: LEFT, Connector_PinSocket_2.54mm:PinSocket_1x12_P2.54mm_Vertical, F.Cu at (102.1, 62.5)
- added J4: RIGHT, Connector_PinSocket_2.54mm:PinSocket_1x12_P2.54mm_Vertical, F.Cu at (147.7, 65.0)
- added R2: 330, Resistor_THT:R_Axial_DIN0207_L6.3mm_D2.5mm_P7.62mm_Horizontal, F.Cu at (133.6, 90.9)
- added R3: 330, Resistor_THT:R_Axial_DIN0207_L6.3mm_D2.5mm_P7.62mm_Horizontal, F.Cu at (128.0, 98.6)
- added R4: 10K, Resistor_THT:R_Axial_DIN0207_L6.3mm_D2.5mm_P7.62mm_Horizontal, F.Cu at (106.7, 85.3)
- added R5: 10K, Resistor_THT:R_Axial_DIN0207_L6.3mm_D2.5mm_P7.62mm_Horizontal, F.Cu at (106.7, 59.9)
- added S1: SW_slide, Connector_PinSocket_2.54mm:PinSocket_1x03_P2.54mm_Vertical, F.Cu at (132.6, 52.8)
- added SW1: USER, Connector_PinSocket_2.54mm:PinSocket_1x03_P2.54mm_Vertical, F.Cu at (112.8, 97.5)
- added SW2: MCLR, Connector_PinSocket_2.54mm:PinSocket_1x03_P2.54mm_Vertical, F.Cu at (106.7, 97.5)
- added U2: 3.3V-AP7381, Package_TO_SOT_THT:TO-92L_Inline, F.Cu at (144.8, 53.8)
- C1: value C -> 1uF; footprint Capacitor_THT:C_Disc_D3.4mm_W2.1mm_P2.50mm -> Capacitor_THT:C_Disc_D5.1mm_W3.2mm_P5.00mm
- D1: value LED -> RED
- R1: value R -> 330
- U1: value AP7384-33V -> PIC32-256B; footprint Package_TO_SOT_THT:TO-92L_Inline -> Package_DIP:DIP-28_W7.62mm_Socket
- moved D1 73.0 mm to (140.5, 68.8), turned to -90 degrees
- moved C1 70.1 mm to (137.7, 55.9), turned to -90 degrees
- moved R1 54.9 mm to (140.7, 59.4), turned to 0 degrees
- moved U1 34.9 mm to (120.4, 59.9), turned to 0 degrees
Connections:
- C1 pad 1: Net-(D1-K) -> /Vin
- C1 pad 2: Net-(C1-Pad2) -> GND
- D1 pad 2: Net-(D1-A) -> +3.3V
- R1 pad 1: Net-(U1-VO) -> Net-(D1-K)
- R1 pad 2: Net-(C1-Pad2) -> GND
- U1 pad 1: Net-(U1-VO) -> /~{MCLR}
- U1 pad 2: Net-(J1-Pin_1) -> /A0
- U1 pad 3: Net-(D1-A) -> /A1
Routing:
- net +3.3V: track 0.00 -> 181.8 mm, vias 0 -> 11
- net /~{MCLR}: track 0.00 -> 47.8 mm, vias 0 -> 3
- net Net-(J2-Pin_1): track 0.00 -> 30.7 mm, vias 0 -> 2
- net /A3: track 0.00 -> 25.9 mm, vias 0 -> 2
- net /YELLOW: track 0.00 -> 22.9 mm, vias 0 -> 4
- net Net-(D3-K): track 0.00 -> 20.4 mm, vias 0 -> 3
- net +5V: track 0.00 -> 19.8 mm, vias 0 -> 3
- net /B15: track 0.00 -> 19.7 mm
- net /B14: track 0.00 -> 19.7 mm
- net /B13: track 0.00 -> 19.7 mm
- net /B12: track 0.00 -> 19.7 mm
- net /B11: track 0.00 -> 19.7 mm
- net /B10: track 0.00 -> 19.7 mm
- net /GREEN: track 0.00 -> 19.3 mm, vias 0 -> 2
- net /USER: track 0.00 -> 18.3 mm, vias 0 -> 3
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- added copper zone on B.Cu, net GND
Other:
- board size 50 x 50 mm -> 154 x 84.1 mm
