File: HW4/HW4/HW4.kicad_sch (KiCad schematic)
At the start: 5 parts, among them J1 Conn_01x12_Pin, U1 AP7384-33V

Commit message: idk what happened lol
Parts:
- removed C1: C, Capacitor_THT:C_Disc_D3.4mm_W2.1mm_P2.50mm, symbol Device:C
- removed D1: LED, LED_THT:LED_D3.0mm, symbol Device:LED
- removed J1: Conn_01x12_Pin, symbol Connector:Conn_01x12_Pin
- removed R1: R, Resistor_THT:R_Axial_DIN0207_L6.3mm_D2.5mm_P7.62mm_Horizontal, symbol Device:R
- removed U1: AP7384-33V, Package_TO_SOT_THT:TO-92L_Inline, symbol ME433-HW4:AP7384-33V
- added J1: Adafruit, symbol Connector:Conn_01x06_Pin
- added J2: Battery, symbol Connector:Conn_01x02_Pin
- added SW1: SW_DPDT_x2, symbol ME433-HW4:SW_DPDT_x2
- added U1: PIC32-256B, symbol ME433-HW4:PIC32-256B
- added U2: 3.3V-AP7381, symbol ME433-HW4:3.3V-AP7381
Connections:
- new net: J1.4 (Pin_4), SW1.1 (A)
- new net: J2.1 (Pin_1), SW1.3 (C)
- new net GND: J1.6 (Pin_6), J2.2 (Pin_2)

Commit message: HW4 Done lawl
Parts:
- added C1, C2, C3, C6: 1uF, Capacitor_THT:C_Disc_D5.1mm_W3.2mm_P5.00mm, symbol Device:C
- added C4, C5: 0.1uF, Capacitor_THT:C_Disc_D3.4mm_W2.1mm_P2.50mm, symbol Device:C
- added D1: RED, LED_THT:LED_D3.0mm, symbol Device:LED
- added D2: YELLOW, LED_THT:LED_D3.0mm, symbol Device:LED
- added D3: GREEN, LED_THT:LED_D3.0mm, symbol Device:LED
- added J3: LEFT, Connector_PinSocket_2.54mm:PinSocket_1x12_P2.54mm_Vertical, symbol Connector:Conn_01x12_Pin
- added J4: RIGHT, Connector_PinSocket_2.54mm:PinSocket_1x12_P2.54mm_Vertical, symbol Connector:Conn_01x12_Pin
- added R1, R2, R3: 330, Resistor_THT:R_Axial_DIN0207_L6.3mm_D2.5mm_P7.62mm_Horizontal, symbol Device:R
- added R4, R5: 10K, Resistor_THT:R_Axial_DIN0207_L6.3mm_D2.5mm_P7.62mm_Horizontal, symbol Device:R
- added SW1: USER, Connector_PinSocket_2.54mm:PinSocket_1x03_P2.54mm_Vertical, symbol Switch:SW_Push
- added SW2: MCLR, Connector_PinSocket_2.54mm:PinSocket_1x03_P2.54mm_Vertical, symbol Switch:SW_Push
- J1: value Adafruit -> CP2102; footprint (none) -> Connector_PinSocket_2.54mm:PinSocket_1x06_P2.54mm_Vertical
- J2: footprint (none) -> Connector_PinSocket_2.54mm:PinSocket_1x02_P2.54mm_Vertical
- S1: renamed from SW1; value SW_DPDT_x2 -> SW_slide; footprint (none) -> Connector_PinSocket_2.54mm:PinSocket_1x03_P2.54mm_Vertical
- U1: footprint (none) -> Package_DIP:DIP-28_W7.62mm_Socket
- U2: footprint (none) -> Package_TO_SOT_THT:TO-92L_Inline
Connections:
- net GND: now also U1.19 (VSS), U1.27 (AVSS), U1.8 (Vss), U2.2 (GND), C1.2, C2.2, C3.2, C4.2, C5.2, C6.2, J3.12 (Pin_12), J4.12 (Pin_12), R1.2, SW1.1, SW2.1
- net +5V: now reaches J1.4 (Pin_4), S1.1 (A)
- net +3.3V: now reaches U2.1 (VO)
- net +3.3V: now also U1.13 (VDD), U1.28 (AVDD), C2.1, C3.1, C4.1, C5.1, D1.2 (A), D2.2 (A), D3.2 (A), J3.11 (Pin_11), J4.11 (Pin_11), R4.1, R5.1
- net Vin: now reaches U2.3 (VI)
- net Vin: now also S1.2 (B), C1.1, J3.10 (Pin_10), J4.10 (Pin_10)
- net ~{MCLR}: now reaches U1.1 (~{MCLR})
- net ~{MCLR}: now also R5.2, SW2.2
- net A3: now reaches U1.10 (A3)
- net A3: now also J3.6 (Pin_6)
- net GREEN: now reaches U1.11 (B4)
- net GREEN: now also J3.7 (Pin_7), R3.2
- net USER: now reaches U1.12 (A4)
- net USER: now also R4.2, SW1.2
- net YELLOW: now reaches U1.14 (B5)
- net YELLOW: now also J3.8 (Pin_8), R2.2
- net B6: now reaches U1.15 (B6)
- net B6: now also J3.9 (Pin_9)
- net B7: now reaches U1.16 (B7)
- net B7: now also J4.9 (Pin_9)
- net B8: now reaches U1.17 (B8)
- net B8: now also J4.8 (Pin_8)
- net B9: now reaches U1.18 (B9)
- net B9: now also J4.7 (Pin_7)
- net A0: now reaches U1.2 (A0)
- net A0: now also J3.1 (Pin_1)
- net at U1.20 (VCAP): now also C6.1
- net B10: now reaches U1.21 (B10)
- net B10: now also J4.6 (Pin_6)
- net B11: now reaches U1.22 (B11)
- net B11: now also J4.5 (Pin_5)
- net B12: now reaches U1.23 (B12)
- net B12: now also J4.4 (Pin_4)
- net B13: now reaches U1.24 (B13)
- net B13: now also J4.3 (Pin_3)
- net B14: now reaches U1.25 (B14)
- net B14: now also J4.2 (Pin_2)
- net B15: now reaches U1.26 (B15)
- net B15: now also J4.1 (Pin_1)
- net A1: now reaches U1.3 (A1)
- net A1: now also J3.2 (Pin_2)
- net B0: now reaches U1.4 (B0)
- net B0: now also J3.3 (Pin_3)
- net B1: now reaches U1.5 (B1)
- net B1: now also J3.4 (Pin_4)
- net B2: now reaches U1.6 (B2)
- net B2: now also J3.5 (Pin_5)
- net U1TX: now reaches U1.7 (B3)
- net U1RX: now reaches U1.9 (A2)
- new net: D3.1 (K), R3.1
- new net: D1.1 (K), R1.1
- new net: D2.1 (K), R2.1
